File: -009_012/Xbox-PMS.kicad_sch (KiCad schematic)
At the start: 139 parts, among them IC1 SIC437BED-T1-GE3, IC2 SIC437BED-T1-GE3, IC3 SIC437BED-T1-GE3, IC4 SIC437BED-T1-GE3, J2 USB_C_Receptacle_USB2.0_16P, J3 Jack-DC, J6 Conn_01x04_Pin, J7 Conn_01x04_Pin, J8 Conn_01x01_Pin, J9 Conn_01x01_Pin, U1 TVS2200DRV, U2 TPS25750, U3 CAT24C512

Commit message: Initial Changes
Updates for the following:

1.) Updated all inductor and capacitance values per equations in datasheet. Should minimize power supply ripple and minimize part cost.
2.) Added AND gate for power good output
3.) Rerouted board for simplicity and noise isolation.
Parts:
- removed C11, C66: 22uF, Capacitor_SMD:C_1210_3225Metric, symbol Device:C_Small
- removed C13, C33, C34, C36, C37, C38, C39, C40, C41, C44, C67, C74, C75, C76, C77, C9: 22uF, Capacitor_SMD:C_0603_1608Metric, symbol Device:C_Small
- removed C23, C25, C28, C72, C73: 47uF, Capacitor_SMD:C_1210_3225Metric, symbol Device:C_Small
- removed C42, C43, C45, C78: 0.1uF, Capacitor_SMD:C_0603_1608Metric, symbol Device:C_Small
- removed C46: 100uF 16V, Capacitor_SMD:C_1210_3225Metric, symbol Device:C_Small
- removed C47: 4.7uF 50V, Capacitor_SMD:C_0805_2012Metric, symbol Device:C_Small
- removed C48, C50, C52, C54, C61: 0.1uF 50V, Capacitor_SMD:C_0402_1005Metric, symbol Device:C_Small
- removed C51, C53: 10uF 16V, Capacitor_SMD:C_0603_1608Metric, symbol Device:C_Small
- removed C55, C56, C57: 10uF 16V, Capacitor_SMD:C_0402_1005Metric, symbol Device:C_Small
- removed C58, C59: 22uF 50V, Capacitor_SMD:C_0805_2012Metric, symbol Device:C_Small
- removed C60: 0.1uF, Capacitor_SMD:C_0402_1005Metric, symbol Device:C_Small
- removed C62, C63: 330pF 16V, Capacitor_SMD:C_0201_0603Metric, symbol Device:C_Small
- removed J2: USB_C_Receptacle_USB2.0_16P, Connector_USB:USB_C_Receptacle_GCT_USB4110, symbol Connector:USB_C_Receptacle_USB2.0_16P
- removed J6: Conn_01x04_Pin, Xbox-Charge:PROG, symbol Connector:Conn_01x04_Pin
- removed J8, J9: Conn_01x01_Pin, TestPoint:TestPoint_Pad_1.5x1.5mm, symbol Connector:Conn_01x01_Pin
- removed JP1: Jumper_2_Open, Jumper:SolderJumper-2_P1.3mm_Open_RoundedPad1.0x1.5mm, symbol Jumper:Jumper_2_Open
- removed R21: 10K, Resistor_SMD:R_0402_1005Metric, symbol Device:R_Small
- removed R22, R23: 2.2K, Resistor_SMD:R_0402_1005Metric, symbol Device:R_Small
- removed TP1, TP10, TP2, TP3, TP4, TP5, TP6, TP7, TP8, TP9: TestPoint, Xbox-PMS:pad, symbol Connector:TestPoint
- removed U1: TVS2200DRV, Package_SON:WSON-6-1EP_2x2mm_P0.65mm_EP1x1.6mm, symbol Power_Protection:TVS2200DRV
- removed U2: TPS25750, Xbox-Charge:TPS25750D, symbol TPS25750D:PTPS25750DRJKT
- removed U3: CAT24C512, Package_SO:SOIC-8_3.9x4.9mm_P1.27mm, symbol Memory_EEPROM:CAT24C512
- added C46, C47, C48: 4.7u, Capacitor_SMD:C_1210_3225Metric, symbol Device:C
- added FET1: AONR21307, DFN8_3x3_EP_AOS, symbol Xbox-PMS:AONR21307
- added H1, H10, H11, H12, H13, H14, H15, H16, H2, H5, H6, H7, H8, H9: MountingHole_Pad, TestPoint:TestPoint_THTPad_2.5x2.5mm_Drill1.2mm, symbol Mechanical:MountingHole_Pad
- added H17, H3, H4: MountingHole, MountingHole:MountingHole_2.2mm_M2, symbol Mechanical:MountingHole
- added J1: GSB1C41110SSHR, Xbox-PMS:AMPHENOL_GSB1C41110SSHR, symbol Xbox-PMS:GSB1C41110SSHR
- added R21: 10, Resistor_SMD:R_0402_1005Metric, symbol Device:R
- added R22: 49.9K, Resistor_SMD:R_0402_1005Metric, symbol Device:R
- added R23: 5.1K, Resistor_SMD:R_0402_1005Metric, symbol Device:R
- added R33, R34: 15K, Resistor_SMD:R_0402_1005Metric, symbol Device:R_Small
- added U1: HUSB238_xxxDD, Package_DFN_QFN:WDFN-10-1EP_3x3mm_P0.5mm_EP1.8x2.5mm, symbol Interface_USB:HUSB238_xxxDD
- added U2: 74VHC21FT, TSSOP14B_TOS, symbol Xbox-PMS:74VHC21FT
- C1, C10, C3, C64, C65, C8: MPN CL32A226KPJNNNE -> (none)
- C12, C14, C16, C68: value 1uF -> 0.1uF; MPN CL05A105KO5NNNC -> (none)
- C15, C17, C18, C69: MPN CL10A475KP8NNNC -> (none)
- C19, C20, C22, C70: MPN GRM155R71H104KE14D -> (none)
- C2: value 22uF -> 10uF; MPN CL32A226KPJNNNE -> (none)
- C21, C24, C26, C27, C29, C32: MPN GRM32EC81A476KE19L -> (none)
- C30, C31, C35: MPN GRM188C61E226ME01J -> (none)
- C4, C5, C6: value 22uF -> 0.1uF; footprint Capacitor_SMD:C_1210_3225Metric -> Capacitor_SMD:C_0402_1005Metric; MPN CL32A226KPJNNNE -> (none)
- C49: value 100uF 16V -> 0.1uF; footprint Capacitor_SMD:C_1210_3225Metric -> Capacitor_SMD:C_0402_1005Metric; MPN GRM32ER61A107ME20L -> (none)
- C7: value 22uF -> 0.1uF; footprint Capacitor_SMD:C_0603_1608Metric -> Capacitor_SMD:C_0402_1005Metric; MPN GRM188C61E226ME01J -> (none)
- C71: value 47uF -> 22uF; footprint Capacitor_SMD:C_1210_3225Metric -> Resistor_SMD:R_0805_2012Metric; MPN GRM32EC81A476KE19L -> (none)
- F1: MPN 0679H5000-01 -> (none)
- IC1, IC2, IC3, IC4: MPN 78-SIC431AED-T1-GE3 -> (none)
- J3: MPN PJ-063AH -> (none)
- J7: MPN 171826-4 -> (none); now not fitted; now left out of the parts list
- L1: value 780nH -> 26uH; footprint Inductor_SMD:L_7.3x7.3_H4.5 -> Xbox-PMS:fch1350-270M; MPN SRP7050TA-1R5M -> (none)
- L2: value 820nH -> 330uH; footprint Inductor_SMD:L_7.3x7.3_H4.5 -> Xbox-PMS:IND_SRN8040TA-331M; MPN SRP7050TA-1R5M -> (none)
- L3: value 780nH -> 10uH; footprint Inductor_SMD:L_7.3x7.3_H4.5 -> Xbox-PMS:MDA1870-100M; MPN SRP7050TA-1R5M -> (none)
- L4: value 820nH -> 42uH; footprint Inductor_SMD:L_7.3x7.3_H4.5 -> Xbox-PMS:IND_ETQ-P4M470KFM_PAN; MPN SRP7050TA-1R5M -> (none)
- R1, R10, R11, R12, R2, R7: MPN CRCW040210K0FKEDC -> (none)
- R13, R16, R19, R31: MPN CRCW04022R20FKED -> (none)
- R14, R17: value 45K -> 15K; MPN P-0402H4502BGTS -> (none)
- R15, R18: MPN ERJ-2RKF2551X -> (none)
- R20: MPN CRCW040218K7FKEDC -> (none)
- R24, R25: value 10K -> 100K; MPN CRCW040210K0FKEDC -> (none)
- R26, R27: value 10K -> 15K; MPN CRCW040210K0FKEDC -> (none)
- R28, R3, R5, R8: MPN AC0402FR-7D100KL -> (none)
- R29, R4, R6, R9: MPN CR0402-FX-4993GLF -> (none)
- R30: MPN ERJ-2RKF4300X -> (none)
- R32: MPN AC0402FR-138K2L -> (none)
Connections:
- net PP5V is gone; now on net GND: C49.1
- net 12V: now also H16.1
- net 3V3SB: now also C49.2, H13.1, R34.1, U2.14; no longer R17.1
- net 3V3SW: now also H14.1, H15.1
- net 5VSW: now also H10.1, H11.1, H12.1, H2.1
- net CCx+: now also J1.A5 (CC1), U1.4 (CC1)
- net CCx-: now also J1.B5 (CC2), U1.5 (CC2)
- net EN: now also R24.2
- net GND: now also C4.1, C5.1, C6.1, C7.1, C46.2, C47.2, C48.2, H5.1, H7.1, H8.1, H9.1, J1.A1_B12 (GND_A), J1.B1_A12 (GND_B), J1.SH1 (SHIELD), J1.SH2 (SHIELD__1), J1.SH3 (SHIELD__2), J1.SH4 (SHIELD__3), U1.11 (GND), U2.7; no longer C4.2, C49.2, C5.2, C6.2, C7.2, R24.2, R25.2, R26.2, R27.2
- net PGOOD: now also H1.1, U2.6; no longer IC1.14 (P_GOOD), IC2.14 (P_GOOD), IC3.14 (P_GOOD), IC4.14 (P_GOOD), R1.1, R10.1, R2.1, R7.1
- net VBUS-IN: now also J1.A4_B9 (VBUS_A), J1.B4_A9 (VBUS_B)
- net VBUS-SAFE: now also C4.2, C5.2, C6.2, C7.2, R25.1, C46.1, C47.1, C48.1, FET1.5 (D), FET1.6 (D), FET1.7 (D), FET1.8 (D); no longer C4.1, C5.1, C6.1, C7.1, F1.2, IC1.19 (EN)
- net at IC2.17 (FB), R12.1: now also R26.2; no longer R14.2
- net ENABLE: now reaches R24.1
- net ENABLE: now also H6.1
- net at R27.1: now also R14.2
- net at R26.1: now also R27.2
- removed net VDD: C12.2, C14.2, C15.2, C16.2, C17.2, C18.2, C68.2, C69.2, IC1.12 (V_DRV), IC1.15 (VDD), IC2.12 (V_DRV), IC2.15 (VDD), IC3.12 (V_DRV), IC3.15 (VDD), IC4.12 (V_DRV), IC4.15 (VDD), R1.2, R10.2, R2.2, R28.2, R29.1, R3.2, R4.1, R5.2, R6.1, R7.2, R8.2, R9.1
- new net: C15.2, IC2.12 (V_DRV)
- new net: FET1.4 (G), R22.2, R23.1
- new net: R23.2, U1.10 (GATE)
- new net: C18.2, IC3.12 (V_DRV)
- new net: C69.2, IC4.12 (V_DRV)
- new net: C17.2, IC1.12 (V_DRV)
- new net: R33.1, R34.2
- new net: R17.1, R33.2
- new net: IC1.19 (EN), R25.2
- new net: R21.2, U1.1 (VIN)
- new net D+: J1.A6 (DP1), U1.2 (D+)
- new net D-: J1.A7 (DN1), U1.3 (D-)
- new net PGOOD_12V: IC4.14 (P_GOOD), R10.1, U2.5
- new net PGOOD_3V3: IC2.14 (P_GOOD), R1.1, U2.4
- new net PGOOD_3V3SB: IC1.14 (P_GOOD), R2.1, U2.2
- new net PGOOD_5V: IC3.14 (P_GOOD), R7.1, U2.1
- new net VBUS-FUSED: F1.2, FET1.1 (S), FET1.2 (S), FET1.3 (S), R21.1, R22.1
- new net VDD_12V: C68.2, IC4.15 (VDD), R10.2, R28.2, R29.1
- new net VDD_3SB: C14.2, IC1.15 (VDD), R2.2, R5.2, R6.1
- new net VDD_3V: C12.2, IC2.15 (VDD), R1.2, R3.2, R4.1
- new net VDD_5V: C16.2, IC3.15 (VDD), R7.2, R8.2, R9.1
- no-connect marks 0 -> 14
Other:
- note added: "HUSB238"
- note removed: "TPS25750D"
- moved on the sheet: C2, C21, C24, C27, C30, R11, R12, R14, R15
